File: Electronics/versions/jt-100-v0.1/jt-100.sch (EAGLE design)
At the start: 20 parts, among them IC1 IC_TC7106/7, IC2 IC_AD8495, T1 PAD_TERMINAL-1.02MM_SQUARE, T2 PAD_TERMINAL-1.02MM_ROUND

Commit message: Added par numbers to the main components.
Parts:
- 7SEG1, 7SEG2, 7SEG3: MPN (none) -> LTS-4817CKR-P; OC_DIGIKEY (none) -> 160-1865-2-ND
- IC1: MPN (none) -> TC7106CKW; OC_DIGIKEY (none) -> TC7106CKW-ND
- IC2: MPN (none) -> AD8495ARMZ; OC_DIGIKEY (none) -> AD8495ARMZ-ND
Changed lines of the file:
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@@
 <?xml version="1.0" encoding="utf-8"?>
 <!DOCTYPE eagle SYSTEM "eagle.dtd">
-<eagle version="6.3">
+<eagle version="7.2.0">
 <drawing>
 <settings>
@@
 <setting verticaltext="up"/>
 </settings>
-<grid distance="0.1" unitdist="inch" unit="inch" style="lines" multiple="1" display="yes" altdistance="0.01" altunitdist="inch" altunit="inch"/>
+<grid distance="0.1" unitdist="inch" unit="inch" style="lines" multiple="1" display="no" altdistance="0.01" altunitdist="inch" altunit="inch"/>
 <layers>
 <layer number="1" name="Top" color="4" fill="1" visible="no" active="no"/>
@@
 <parts>
 <part name="U$1" library="dp_devices.v6" deviceset="FRAME_DINA4_L" device=""/>
-<part name="IC1" library="dp_devices.v6" deviceset="IC_TC7106/7" device=""/>
-<part name="IC2" library="dp_devices.v6" deviceset="IC_AD8495" device=""/>
+<part name="IC1" library="dp_devices.v6" deviceset="IC_TC7106/7" device="">
+<attribute name="MPN" value="TC7106CKW"/>
+<attribute name="OC_DIGIKEY" value="TC7106CKW-ND"/>
+</part>
+<part name="IC2" library="dp_devices.v6" deviceset="IC_AD8495" device="">
+<attribute name="MPN" value="AD8495ARMZ"/>
+<attribute name="OC_DIGIKEY" value="AD8495ARMZ-ND"/>
+</part>
 <part name="VCC1" library="dp_devices.v6" deviceset="SUPPLY_VCC" device=""/>
 <part name="GND1" library="dp_devices.v6" deviceset="SUPPLY_GND" device=""/>
@@
 <part name="C3" library="dp_devices.v6" deviceset="CAPACITOR_NPOL" device="-1206"/>
 <part name="C4" library="dp_devices.v6" deviceset="CAPACITOR_NPOL" device="-1206"/>
-<part name="7SEG1" library="dp_devices.v6" deviceset="DISP_7SEG" device="-10MM" value="DISP_7SEG-10MM"/>
-<part name="7SEG2" library="dp_devices.v6" deviceset="DISP_7SEG" device="-10MM" value="DISP_7SEG-10MM"/>
-<part name="7SEG3" library="dp_devices.v6" deviceset="DISP_7SEG" device="-10MM" value="DISP_7SEG-10MM"/>
+<part name="7SEG1" library="dp_devices.v6" deviceset="DISP_7SEG" device="-10MM" value="DISP_7SEG-10MM">
+<attribute name="MPN" value="LTS-4817CKR-P"/>
+<attribute name="OC_DIGIKEY" value="160-1865-2-ND"/>
+</part>
+<part name="7SEG2" library="dp_devices.v6" deviceset="DISP_7SEG" device="-10MM" value="DISP_7SEG-10MM">
+<attribute name="MPN" value="LTS-4817CKR-P"/>
+<attribute name="OC_DIGIKEY" value="160-1865-2-ND"/>
+</part>
+<part name="7SEG3" library="dp_devices.v6" deviceset="DISP_7SEG" device="-10MM" value="DISP_7SEG-10MM">
+<attribute name="MPN" value="LTS-4817CKR-P"/>
+<attribute name="OC_DIGIKEY" value="160-1865-2-ND"/>
+</part>
 <part name="R5" library="dp_devices.v6" deviceset="RESISTOR" device="-1206" value="5.1R 1/4W"/>
 <part name="VCC4" library="dp_devices.v6" deviceset="SUPPLY_VCC" device=""/>
@@
 <instance part="U$1" gate="G$1" x="0" y="0"/>
 <instance part="U$1" gate="G$2" x="158.75" y="3.81"/>
-<instance part="IC1" gate="IC" x="91.44" y="76.2"/>
-<instance part="IC2" gate="IC" x="33.02" y="101.6"/>
+<instance part="IC1" gate="IC" x="91.44" y="76.2">
+<attribute name="OC_DIGIKEY" x="91.44" y="76.2" size="1.778" layer="96" display="off"/>
+<attribute name="MPN" x="91.44" y="76.2" size="1.778" layer="96" display="off"/>
+</instance>
+<instance part="IC2" gate="IC" x="33.02" y="101.6">
+<attribute name="OC_DIGIKEY" x="33.02" y="101.6" size="1.778" layer="96" display="off"/>
+<attribute name="MPN" x="33.02" y="101.6" size="1.778" layer="96" display="off"/>
+</instance>
 <instance part="VCC1" gate="SUP" x="25.4" y="116.84"/>
 <instance part="GND1" gate="G$1" x="25.4" y="83.82" smashed="yes"/>
@@
 <attribute name="VALUE" x="68.58" y="81.28" size="1.778" layer="96" rot="R90"/>
 </instance>
-<instance part="7SEG1" gate="DISP" x="149.86" y="134.62"/>
-<instance part="7SEG2" gate="DISP" x="182.88" y="134.62"/>
-<instance part="7SEG3" gate="DISP" x="215.9" y="134.62"/>
+<instance part="7SEG1" gate="DISP" x="149.86" y="134.62">
+<attribute name="MPN" x="149.86" y="134.62" size="1.778" layer="96" display="off"/>
+<attribute name="OC_DIGIKEY" x="149.86" y="134.62" size="1.778" layer="96" display="off"/>
+</instance>
+<instance part="7SEG2" gate="DISP" x="182.88" y="134.62">
+<attribute name="MPN" x="182.88" y="134.62" size="1.778" layer="96" display="off"/>
+<attribute name="OC_DIGIKEY" x="182.88" y="134.62" size="1.778" layer="96" display="off"/>
+</instance>
+<instance part="7SEG3" gate="DISP" x="215.9" y="134.62">
+<attribute name="MPN" x="215.9" y="134.62" size="1.778" layer="96" display="off"/>
+<attribute name="OC_DIGIKEY" x="215.9" y="134.62" size="1.778" layer="96" display="off"/>
+</instance>
 <instance part="R5" gate="R" x="137.16" y="160.02" smashed="yes" rot="R90">
 <attribute name="NAME" x="139.7" y="160.02" size="1.778" layer="95" font="vector"/>
